Commit message: temp

File: hex_zmq_servers/robot/hexarm/urdf/archer_y6/empty.urdf (robot description, URDF)
Before this commit: robot archer_y6, 7 links, 6 joints
Joints:
- joint joint_2: origin xyz=0.0199999999999999 0 0.0450000000000004 rpy=0 0 0 -> xyz=0.02 0 0.045 rpy=0 0 0
- joint joint_4: origin xyz=-0.0599999999999998 0 0.245 rpy=0 0 0 -> xyz=-0.06 0 0.245 rpy=0 0 0
- joint joint_5: origin xyz=-0.0553005693392305 0 0.0702500000000025 rpy=0 0 0 -> xyz=-0.0553 0 0.070 rpy=0 0 0
- joint joint_6: origin xyz=0.0578000000000073 0 0.0289500000000001 rpy=0 0 0 -> xyz=0.0553 0 0.029 rpy=0 0 0

File: hex_zmq_servers/robot/hexarm/urdf/archer_y6/gp100.urdf (robot description, URDF)
Before this commit: robot archer_y6, 7 links, 6 joints
Joints:
- joint joint_2: origin xyz=0.0199999999999999 0 0.0450000000000004 rpy=0 0 0 -> xyz=0.02 0 0.045 rpy=0 0 0
- joint joint_4: origin xyz=-0.0599999999999998 0 0.245 rpy=0 0 0 -> xyz=-0.06 0 0.245 rpy=0 0 0
- joint joint_5: origin xyz=-0.0553005693392305 0 0.0702500000000025 rpy=0 0 0 -> xyz=-0.0553 0 0.070 rpy=0 0 0
- joint joint_6: origin xyz=0.0578000000000073 0 0.0289500000000001 rpy=0 0 0 -> xyz=0.0553 0 0.029 rpy=0 0 0

File: hex_zmq_servers/robot/hexarm/urdf/archer_y6/gp100_handle.urdf (robot description, URDF)
Before this commit: robot archer_y6, 7 links, 6 joints
Joints:
- joint joint_2: origin xyz=0.0199999999999999 0 0.0450000000000004 rpy=0 0 0 -> xyz=0.02 0 0.045 rpy=0 0 0
- joint joint_4: origin xyz=-0.0599999999999998 0 0.245 rpy=0 0 0 -> xyz=-0.06 0 0.245 rpy=0 0 0
- joint joint_5: origin xyz=-0.0553005693392305 0 0.0702500000000025 rpy=0 0 0 -> xyz=-0.0553 0 0.070 rpy=0 0 0
- joint joint_6: origin xyz=0.0578000000000073 0 0.0289500000000001 rpy=0 0 0 -> xyz=0.0553 0 0.029 rpy=0 0 0

File: hex_zmq_servers/robot/hexarm/urdf/archer_y6/gp100_p050.urdf (robot description, URDF)
Before this commit: robot archer_y6, 7 links, 6 joints
Joints:
- joint joint_2: origin xyz=0.0199999999999999 0 0.0450000000000004 rpy=0 0 0 -> xyz=0.02 0 0.045 rpy=0 0 0
- joint joint_4: origin xyz=-0.0599999999999998 0 0.245 rpy=0 0 0 -> xyz=-0.06 0 0.245 rpy=0 0 0
- joint joint_5: origin xyz=-0.0553005693392305 0 0.0702500000000025 rpy=0 0 0 -> xyz=-0.0553 0 0.070 rpy=0 0 0
- joint joint_6: origin xyz=0.0578000000000073 0 0.0289500000000001 rpy=0 0 0 -> xyz=0.0553 0 0.029 rpy=0 0 0

File: hex_zmq_servers/robot/hexarm/urdf/archer_y6/gp100_p050_handle.urdf (robot description, URDF)
Before this commit: robot archer_y6, 7 links, 6 joints
Joints:
- joint joint_2: origin xyz=0.0199999999999999 0 0.0450000000000004 rpy=0 0 0 -> xyz=0.02 0 0.045 rpy=0 0 0
- joint joint_4: origin xyz=-0.0599999999999998 0 0.245 rpy=0 0 0 -> xyz=-0.06 0 0.245 rpy=0 0 0
- joint joint_5: origin xyz=-0.0553005693392305 0 0.0702500000000025 rpy=0 0 0 -> xyz=-0.0553 0 0.070 rpy=0 0 0
- joint joint_6: origin xyz=0.0578000000000073 0 0.0289500000000001 rpy=0 0 0 -> xyz=0.0553 0 0.029 rpy=0 0 0
